File: aqkitty!/hrsens.kicad_pcb (KiCad board)
At the start: 2 copper layers, 69.8 x 97.9 mm, 16 parts, among them U1 ENS160-BGLM, U2 XIAO-RP2040-DIP, U3 OLED_0.91_128x32, U4 SHT30-DIS

Commit message: umm extra files
i think they got left behind idk. check last commit
Parts:
- moved C1 67.2 mm to (94.0, 126.8), turned to 180 degrees
- moved D1 51.2 mm to (119.8, 132.0)
- moved R2 44.1 mm to (79.0, 123.3)
- moved U4 44.0 mm to (130.6, 127.8)
- moved R1 43.5 mm to (79.1, 127.6)
- moved R3 42.8 mm to (124.3, 132.1)
- moved U1 41.0 mm to (131.4, 116.5), turned to -90 degrees
- moved C3 40.1 mm to (126.4, 127.8), turned to 180 degrees
- moved C2 34.5 mm to (126.6, 118.0), turned to 180 degrees
Connections:
- D1 pad 1: GND -> Net-(D1-A)
- R3 pad 1: Net-(D1-A) -> GND
- R3 pad 2: Net-(U2-GPIO26/ADC0/A0) -> Net-(D1-A)
- U2 pad 1: Net-(U2-GPIO26/ADC0/A0) -> Net-(D1-A)
Routing:
- net /SDA: track 0.00 -> 127.6 mm
- net +3V3: track 0.00 -> 115.0 mm, vias 0 -> 1
- net /SCL: track 0.00 -> 103.5 mm, vias 0 -> 2
- net GND: track 0.00 -> 77.6 mm, vias 0 -> 13
- net Net-(D1-A): track 0.00 -> 15.9 mm, vias 0 -> 1
- added copper zone on B.Cu, net GND
- added copper zone on F.Cu, net GND
